File: Hardware/SmartWatchPCB.brd (EAGLE design)
At the start: 46 x 35 mm, 105 parts, among them IC1 BQ25180YBGR, IC2 DRV2605YZFR, IC3 BMA423_BMA423, IC9 RT6160AWSC, J1 503480-2400, J2 TC2030-IDC, J4 KH-TYPE-C-16P, Q1 20V/4.2A/52mΩ/1.4W, Q3 SI1308EDL-T1-GE3, U1 NRF52840_QF, U3 MAX17048G+T10, X1 32MHz, X2 32.768kHz

Commit message: blyat
Parts:
- EPD_C1, EPD_C10, EPD_C11, EPD_C12, EPD_C2, EPD_C6, EPD_C7, EPD_C8, EPD_C9: value 0.1uF/50V -> 1uF/50V; device InkTime_v5:NORDIC_NRF_3_RESC0201_L -> InkTime_v5:NORDIC_NRF_3_RESC0402_L
- L2, L3: device InkTime_v5:MLP2016SR47MT0S1_INDC2016X100N -> InkTime_v5:NORDIC_NRF_2_RESC0201_L
- L5: value 68uH -> 48uH; device InkTime_v5:NORDIC_NRF_2_RESC0402_L -> InkTime_v5:ESP32_C6_LIBRARY_2_IND_4828-WE-TPC_WRE
- moved TP_3.3V 60.9 mm to (15.6, 16.1)
- moved TP_GND 51.9 mm to (21.5, 10.4)
- moved C27 45.1 mm to (18.1, 11.7), turned to 180 degrees
- moved TP_SCL 43.3 mm to (18.1, 15.3)
- moved U3 41.5 mm to (17.6, 9.60), turned to 270 degrees
- moved TP_VREG 41.0 mm to (5.10, 9.60)
- moved TP_VBAT 38.2 mm to (20.5, 13.7)
- moved IC2 38.1 mm to (-18.1, -11.5), turned to 180 degrees
- moved C34 38.1 mm to (-18.1, -10.0), turned to 270 degrees
- moved C32 37.7 mm to (-17.9, -12.8), turned to 180 degrees
- moved TP_SDA 35.8 mm to (21.5, 7.50)
- moved TP_SWDIO 33.5 mm to (-6.70, 1.60)
- moved TP_SWDCLK 31.5 mm to (-4.70, 3.50)
- moved TP_RESET 26.2 mm to (-2.00, 1.70)
- moved TP_3V3 24.2 mm to (-7.70, -9.00)
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Connections:
- removed net ALERT/2.5C: U1.P$J24
- removed net N$10: C19.1, IC3.10, IC3.7
- removed net N$14: IC3.12
- removed net N$19: C5.2
- removed net N$33: D4.1
- removed net N$34: D2.2
- removed net N$35: D5.1
- removed net N$37: C12.1, U1.P$A22
- removed net N$38: TP_VBAT.TP
- removed net N$40: TP_OP.TP
- removed net N$43: J1.9
- removed net N$44: J1.10
- removed net N$45: J1.11
- removed net N$47: J1.12
- removed net N$48: J1.13
- removed net N$49: J1.14
- removed net N$50: EPD_C5.1, J1.15, J1.16
- removed net N$53: IC2.A3
- removed net N$54: J4.B7
- removed net N$55: J4.B6
- removed net N$56: IC2.C3
- removed net N$6: IC3.2
- removed net N$60: J4.A7
- removed net N$61: J4.A6
- removed net N$63: J4.A4_B9, J4.A9_B4
- removed net N$7: IC3.3
- removed net SDL: U3.8
- new net OUT+: IC2.A3, TP_OP.TP
- net 3V3: now also C12.1, C19.1, IC3.10, IC3.3, IC3.7, U1.P$A22
- net ALERT: now also U1.P$J24
- net DN: now also J4.A7, J4.B7
- net DP: now also J4.A6, J4.B6
- net EPD_3V3: now also EPD_C5.1, J1.15, J1.16, L5.2; no longer L5.1
- net EPD_BUSY: now also J1.9
- net EPD_CS: now also J1.12
- net EPD_DC: now also J1.11
- net EPD_RST: now also J1.10
- net GND: now also C5.2, D4.1
- net MOSI: now also J1.14
- net N$31: now also L5.1; no longer L5.2
- net OUT-: now also IC2.C3
- net PREVGH: now also D5.1
- net PREVGL: now also D2.2
- net SCK: now also J1.13
- net SCL: now also IC3.12
- net SDA: now also IC3.2, U3.8
- net VBAT: now also TP_VBAT.TP
- net VBUS: now also J4.A4_B9, J4.A9_B4
Routing:
- net 3V3: track 0.00 -> 168.5 mm, vias 0 -> 11
- net SCL: track 0.00 -> 101.1 mm, vias 0 -> 6
- net SDA: track 0.00 -> 96.3 mm, vias 0 -> 9
- net HAPTIC_EN: track 0.00 -> 78.5 mm, vias 0 -> 6
- net EPD_CS: track 0.00 -> 62.6 mm, vias 0 -> 6
- net MOSI: track 0.00 -> 58.4 mm, vias 0 -> 4
- net SCK: track 0.00 -> 56.4 mm, vias 0 -> 2
- net GND: track 0.00 -> 44.3 mm, vias 0 -> 53
- net P1.01: track 0.00 -> 43.7 mm, vias 0 -> 4
- net P0.13: track 1.27 -> 29.9 mm, vias 0 -> 4
- net VBUS: track 0.00 -> 28.6 mm
- net SWDIO: track 0.00 -> 28.4 mm, vias 0 -> 2
- net SWDCLK: track 0.00 -> 28.4 mm, vias 0 -> 2
- net N$24: track 0.00 -> 28.0 mm, vias 0 -> 2
- net EPD_RST: track 0.00 -> 27.7 mm, vias 0 -> 4
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- added copper zone on layer 1, net GND
- added copper zone on layer 16, net GND
- added copper zone on layer 2, net GND
Other:
- outline, holes or cut-outs redrawn
